File: AMP/AMP.kicad_pcb (KiCad board)
At the start: 2 copper layers, 125 parts, among them U1 NE5532, U10 NE5532, U11 NE5532, U12 NE5532, U13 NE5532, U14 NE5532, U15 NE5532, U16 NE5532, U17 NE5532, U18 NE5532, U2 NE5532, U3 NE5532, U4 NE5532, U5 NE5532, U6 NE5532, U7 NE5532, U8 NE5532, U9 NE5532

Commit message: amp updated files
Parts:
- added J1: AudioJack4, Connector_Audio:Jack_3.5mm_PJ320D_Horizontal, F.Cu at (171.4, -21.6)
- added J2: Screw_Terminal_01x02, TerminalBlock:TerminalBlock_Altech_AK300-2_P5.00mm, F.Cu at (142.0, -24.1)
- added J3: AudioJack4, Connector_Audio:Jack_3.5mm_PJ320D_Horizontal, F.Cu at (133.3, 233.7)
- moved C20 194.3 mm to (256.5, 104.1)
- moved C18 185.4 mm to (247.8, 114.3)
- moved U4 170.9 mm to (271.8, 101.6)
- moved C26 165.3 mm to (35.7, 170.4)
- moved C27 163.3 mm to (20.3, 176.4)
- moved R44 161.9 mm to (45.7, 172.7)
- moved R15 156.7 mm to (258.2, 57.3)
- moved R42 156.4 mm to (266.7, 96.5)
- moved C31 151.4 mm to (199.6, 132.1)
- moved R10 150.8 mm to (265.8, 57.3)
- moved R12 149.6 mm to (264.2, 67.3)
- moved R26 141.0 mm to (265.8, 49.7)
- moved R48 140.8 mm to (62.0, 180.3)
- moved C15 140.0 mm to (31.9, 22.9)
- moved R16 139.5 mm to (248.0, 67.4)
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Connections:
- C13 pad 1: Net-(C13-Pad1) -> +15V
- C13 pad 2: Net-(C13-Pad2) -> GND
- C14 pad 1: Net-(C14-Pad1) -> +15V
- C14 pad 2: Net-(C14-Pad2) -> GND
- C15 pad 1: Net-(C15-Pad1) -> +15V
- C15 pad 2: Net-(C15-Pad2) -> GND
- C16 pad 1: Net-(C16-Pad1) -> +15V
- C16 pad 2: Net-(C16-Pad2) -> GND
- C21 pad 1: Net-(C21-Pad1) -> +15V
- C21 pad 2: Net-(C21-Pad2) -> GND
- C22 pad 1: Net-(C22-Pad1) -> +15V
- C22 pad 2: Net-(C22-Pad2) -> GND
- C26 pad 1: Net-(C26-Pad1) -> +15V
- C26 pad 2: Net-(C26-Pad2) -> GND
- C27 pad 1: Net-(C27-Pad1) -> +15V
- C27 pad 2: Net-(C27-Pad2) -> GND
- C28 pad 1: Net-(C28-Pad1) -> +15V
- C28 pad 2: Net-(C28-Pad2) -> GND
- C29 pad 1: Net-(C29-Pad1) -> +15V
- C29 pad 2: Net-(C29-Pad2) -> GND
- C30 pad 1: Net-(C30-Pad1) -> +15V
- C30 pad 2: Net-(C30-Pad2) -> GND
- C32 pad 1: Net-(C32-Pad1) -> +15V
- C32 pad 2: Net-(C32-Pad2) -> GND
- C33 pad 1: Net-(C33-Pad1) -> +15V
- C33 pad 2: Net-(C33-Pad2) -> GND
- C34 pad 1: Net-(C34-Pad1) -> +15V
- C34 pad 2: Net-(C34-Pad2) -> GND
- C35 pad 1: Net-(C35-Pad1) -> +15V
- C35 pad 2: Net-(C35-Pad2) -> GND
- C36 pad 1: Net-(C36-Pad1) -> +15V
- C36 pad 2: Net-(C36-Pad2) -> GND
- C7 pad 1: Net-(C7-Pad1) -> +15V
- C7 pad 2: Net-(C7-Pad2) -> GND
- C8 pad 1: Net-(C8-Pad1) -> +15V
- C8 pad 2: Net-(C8-Pad2) -> GND
- U1 pad 4: Net-(C7-Pad2) -> GND
- U1 pad 8: Net-(C7-Pad1) -> +15V
- U10 pad 4: Net-(C27-Pad2) -> GND
- U10 pad 8: Net-(C27-Pad1) -> +15V
- U11 pad 4: Net-(C28-Pad2) -> GND
- U11 pad 8: Net-(C28-Pad1) -> +15V
- U12 pad 4: Net-(C29-Pad2) -> GND
- U12 pad 8: Net-(C29-Pad1) -> +15V
- U13 pad 4: Net-(C30-Pad2) -> GND
- U13 pad 8: Net-(C30-Pad1) -> +15V
- U14 pad 4: Net-(C32-Pad2) -> GND
- U14 pad 8: Net-(C32-Pad1) -> +15V
- U15 pad 4: Net-(C33-Pad2) -> GND
- U15 pad 8: Net-(C33-Pad1) -> +15V
- U16 pad 4: Net-(C34-Pad2) -> GND
- U16 pad 8: Net-(C34-Pad1) -> +15V
- U17 pad 4: Net-(C35-Pad2) -> GND
- U17 pad 8: Net-(C35-Pad1) -> +15V
- U18 pad 4: Net-(C36-Pad2) -> GND
- U18 pad 8: Net-(C36-Pad1) -> +15V
- U2 pad 4: Net-(C8-Pad2) -> GND
- U2 pad 8: Net-(C8-Pad1) -> +15V
- U3 pad 4: Net-(C21-Pad2) -> GND
- U3 pad 8: Net-(C21-Pad1) -> +15V
- U4 pad 4: Net-(C22-Pad2) -> GND
- U4 pad 8: Net-(C22-Pad1) -> +15V
- U5 pad 4: Net-(C15-Pad2) -> GND
- U5 pad 8: Net-(C15-Pad1) -> +15V
- U6 pad 4: Net-(C16-Pad2) -> GND
- U6 pad 8: Net-(C16-Pad1) -> +15V
- U7 pad 4: Net-(C13-Pad2) -> GND
- U7 pad 8: Net-(C13-Pad1) -> +15V
- U8 pad 4: Net-(C14-Pad2) -> GND
- U8 pad 8: Net-(C14-Pad1) -> +15V
- U9 pad 4: Net-(C26-Pad2) -> GND
- U9 pad 8: Net-(C26-Pad1) -> +15V

Commit message: pcb layout
Parts:
- R1, R2, R8, R9: footprint Resistor_THT:R_Axial_DIN0516_L15.5mm_D5.0mm_P20.32mm_Horizontal -> Resistor_SMD:R_0603_1608Metric
- moved R20 61.3 mm to (130.4, 56.6), turned to -90 degrees
- moved R6 58.1 mm to (128.1, 56.6), turned to -90 degrees
- moved C8 52.5 mm to (142.1, 53.3)
- moved R8 48.0 mm to (143.6, 50.2), turned to 90 degrees
- moved U2 46.1 mm to (135.9, 55.4)
- moved R19 43.2 mm to (130.4, 50.3), turned to -90 degrees
- moved C3 42.5 mm to (145.9, 56.6), turned to 90 degrees
- moved C2 41.8 mm to (145.9, 50.2), turned to 90 degrees
- moved R5 38.6 mm to (128.1, 50.3), turned to -90 degrees
- moved R1 37.6 mm to (141.4, 50.2), turned to -90 degrees
- moved R9 26.6 mm to (143.6, 56.6), turned to 90 degrees
- moved R2 21.6 mm to (141.4, 56.6), turned to -90 degrees
- moved J1 19.7 mm to (152.4, -26.7), turned to -90 degrees
- moved U1 16.5 mm to (135.9, 48.9)
- moved C7 10.7 mm to (142.1, 46.9)
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Connections:
- J1 pad R1: LEFT_AUDIO_IN -> RIGHT_AUDIO_IN
- J1 pad T: RIGHT_AUDIO_IN -> LEFT_AUDIO_IN
Routing:
- net Net-(C3-Pad1): track 0.00 -> 13.1 mm
- net Net-(C2-Pad1): track 0.00 -> 13.1 mm
- net GND: track 0.00 -> 10.2 mm
- net Net-(R19-Pad1): track 0.00 -> 8.40 mm
- net Net-(R20-Pad1): track 0.00 -> 8.35 mm
- net Net-(R5-Pad1): track 0.00 -> 5.78 mm
- net Net-(R6-Pad1): track 0.00 -> 5.73 mm
- net +15V: track 0.00 -> 5.49 mm
- net VBIAS_R: track 0.00 -> 2.29 mm
- net VBIAS_L: track 0.00 -> 2.29 mm

Commit message: updated files
Parts:
- removed C27, C35: 100n, Resistor_SMD:R_0603_1608Metric
- removed C38: 2200u, Capacitor_THT:CP_Radial_D12.5mm_P5.00mm
- removed R44, R51, R59, R63: 1, Resistor_SMD:R_1206_3216Metric
- removed R65: 10, Resistor_SMD:R_0603_1608Metric
- removed U17, U18, U9: NE5532, AUDIO_ECAD:NE5532DR
- added C39: 100n, Resistor_SMD:R_0603_1608Metric, F.Cu at (134.9, 96.0)
- added C40: 100n, Resistor_SMD:R_0603_1608Metric, F.Cu at (134.9, 103.9)
- added C41: 100n, Resistor_SMD:R_0603_1608Metric, F.Cu at (134.9, 111.7)
- added C42: 100n, Resistor_SMD:R_0603_1608Metric, F.Cu at (140.4, 83.7)
- added C43: 100n, Resistor_SMD:R_0603_1608Metric, F.Cu at (141.1, 107.4)
- added C44: 100n, Resistor_SMD:R_0603_1608Metric, F.Cu at (141.1, 99.5)
- added C45: 100n, Resistor_SMD:R_0603_1608Metric, F.Cu at (141.1, 91.6)
- added J4: Barrel_Jack_MountingPin, Connector_BarrelJack:BarrelJack_Horizontal, F.Cu at (112.0, 58.0)
- added R69: 10, Resistor_SMD:R_0603_1608Metric, F.Cu at (130.0, 87.8)
- added R70: 10, Resistor_SMD:R_0603_1608Metric, F.Cu at (137.2, 112.5)
- added R71: 10k, Resistor_SMD:R_1206_3216Metric, F.Cu at (120.5, 107.2)
- added R73: 1, Resistor_SMD:R_1206_3216Metric, F.Cu at (135.7, 93.8)
- added R74: 1, Resistor_SMD:R_1206_3216Metric, F.Cu at (135.7, 101.7)
- added R75: 1, Resistor_SMD:R_1206_3216Metric, F.Cu at (135.7, 109.6)
- added R76: 10, Resistor_SMD:R_0603_1608Metric, F.Cu at (128.2, 87.8)
- added R77: 1, Resistor_SMD:R_1206_3216Metric, F.Cu at (140.3, 112.1)
- added R78: 1, Resistor_SMD:R_1206_3216Metric, F.Cu at (140.3, 104.2)
- added R79: 1, Resistor_SMD:R_1206_3216Metric, F.Cu at (140.3, 96.3)
- added R81: 1, Resistor_SMD:R_1206_3216Metric, F.Cu at (140.3, 109.5)
- added R82: 1, Resistor_SMD:R_1206_3216Metric, F.Cu at (140.3, 101.7)
- added R83: 1, Resistor_SMD:R_1206_3216Metric, F.Cu at (140.3, 93.8)
- added REF**: MountingHole_2.2mm_M2_Pad_Via, MountingHole:MountingHole_2.2mm_M2_Pad_Via, F.Cu at (78.5, 51.5)
- added REF**: MountingHole_2.2mm_M2_Pad_Via, MountingHole:MountingHole_2.2mm_M2_Pad_Via, F.Cu at (181.5, 116.5)
- added REF**: MountingHole_2.2mm_M2_Pad_Via, MountingHole:MountingHole_2.2mm_M2_Pad_Via, F.Cu at (181.5, 51.5)
- added REF**: MountingHole_2.2mm_M2_Pad_Via, MountingHole:MountingHole_2.2mm_M2_Pad_Via, F.Cu at (78.5, 116.5)
- added U19: NE5532, AUDIO_ECAD:NE5532DR, F.Cu at (130.3, 93.8)
- added U20: NE5532, AUDIO_ECAD:NE5532DR, F.Cu at (130.3, 101.7)
- added U21: NE5532, AUDIO_ECAD:NE5532DR, F.Cu at (130.3, 109.6)
- added U22: NE5532, AUDIO_ECAD:NE5532DR, F.Cu at (134.8, 86.5)
- added U23: NE5532, AUDIO_ECAD:NE5532DR, F.Cu at (145.6, 109.5)
- added U24: NE5532, AUDIO_ECAD:NE5532DR, F.Cu at (145.6, 101.7)
- added U25: NE5532, AUDIO_ECAD:NE5532DR, F.Cu at (145.6, 93.8)
- C1: value 220u -> 10u; footprint Capacitor_THT:CP_Radial_D6.3mm_P2.50mm -> Resistor_SMD:R_0603_1608Metric
- C10, C23, C24, C9: value 100p -> 100n
- C21, C22, C7, C8: value 100n -> 100p
- C26: value 100n -> 2200u; footprint Resistor_SMD:R_0603_1608Metric -> Capacitor_THT:CP_Radial_D12.5mm_P5.00mm
- C3: value 10u -> 220u; footprint Resistor_SMD:R_0603_1608Metric -> Capacitor_THT:CP_Radial_D6.3mm_P2.50mm
- C31: value 10u -> 100n; footprint Capacitor_THT:C_Axial_L22.0mm_D10.5mm_P27.50mm_Horizontal -> Resistor_SMD:R_0603_1608Metric
- C36: value 100n -> 10u; footprint Resistor_SMD:R_0603_1608Metric -> Capacitor_THT:C_Axial_L22.0mm_D10.5mm_P27.50mm_Horizontal
- J2: value Screw_Terminal_01x02 -> AudioJack4; footprint TerminalBlock:TerminalBlock_Altech_AK300-2_P5.00mm -> Connector_Audio:Jack_3.5mm_PJ320D_Horizontal
- J3: value AudioJack4 -> Screw_Terminal_01x02; footprint Connector_Audio:Jack_3.5mm_PJ320D_Horizontal -> TerminalBlock:TerminalBlock_bornier-2_P5.08mm
- R18: value 47k -> 10
- R20: value 10 -> 47k
- R27, R28: value 22k -> 1k
- R29: value 1k -> 10
- R30: value 100 -> 10
- R31: value 100 -> 22k
- R32: value 1k -> 22k
- R33, R34: value 10 -> 100
- R35, R36: value 10 -> 5.6k
- R37, R38: value 22k -> 10
- R39, R40: value 5.6k -> 22k
- R46, R57, R60, R67: value 10 -> 1; footprint Resistor_SMD:R_0603_1608Metric -> Resistor_SMD:R_1206_3216Metric
- R48, R55: value 1 -> 10; footprint Resistor_SMD:R_1206_3216Metric -> Resistor_SMD:R_0603_1608Metric
- R50, R64: value 1 -> 10k
- R54, R66, R68: value 10k -> 1
- R7: value 3.3k -> 2.2k; footprint Resistor_SMD:R_1206_3216Metric -> Resistor_SMD:R_0603_1608Metric
- R9: value 2.2k -> 3.3k; footprint Resistor_SMD:R_0603_1608Metric -> Resistor_SMD:R_1206_3216Metric
- RV1: footprint Potentiometer_THT:Potentiometer_Alpha_RD902F-40-00D_Dual_Vertical -> Potentiometer_THT:Potentiometer_Alps_RK163_Dual_Horizontal
- moved R35 183.8 mm to (81.7, 76.8), turned to 90 degrees
- moved J3 178.8 mm to (126.0, 55.0), turned to 180 degrees
- moved C10 172.4 mm to (89.9, 59.0), turned to 180 degrees
- moved R18 160.7 mm to (82.3, 57.1), turned to 180 degrees
- moved C14 156.1 mm to (92.1, 76.1)
- moved C13 143.4 mm to (92.1, 69.4)
- moved C34 142.2 mm to (90.2, 91.5), turned to 180 degrees
- moved R34 138.6 mm to (171.1, 70.2), turned to -90 degrees
- moved U4 138.1 mm to (137.1, 71.3)
- moved C17 138.0 mm to (158.5, 75.0), turned to -90 degrees
- moved C23 138.0 mm to (161.3, 57.1)
- moved R39 137.4 mm to (163.8, 71.4), turned to 180 degrees
- moved J2 136.7 mm to (112.8, 113.8), turned to 90 degrees
- moved R28 135.2 mm to (128.7, 76.8), turned to 90 degrees
- moved RV1 134.9 mm to (156.0, 109.5), turned to 90 degrees
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Connections:
- C1 pad 1: LEFT_BUF_AUDIO -> Net-(C1-Pad1)
- C1 pad 2: L_Pot1 -> GND
- C10 pad 1: Net-(C10-Pad1) -> +15V
- C10 pad 2: VOL_OUT_R -> GND
- C21 pad 1: +15V -> Net-(C21-Pad1)
- C21 pad 2: GND -> Net-(C21-Pad2)
- C22 pad 1: +15V -> Net-(C22-Pad1)
- C22 pad 2: GND -> Net-(C22-Pad2)
- C23 pad 1: Net-(C23-Pad1) -> +15V
- C23 pad 2: Net-(C23-Pad2) -> GND
- C24 pad 1: Net-(C24-Pad1) -> +15V
- C24 pad 2: Net-(C24-Pad2) -> GND
- C26 pad 1: +15V -> Net-(C26-Pad1)
- C26 pad 2: GND -> AUDIO_OUT_L
- C3 pad 1: Net-(C3-Pad1) -> LEFT_BUF_AUDIO
- C3 pad 2: GND -> L_Pot1
- C31 pad 1: VOL_OUT_R -> +15V
- C31 pad 2: Net-(C31-Pad2) -> GND
- C36 pad 1: +15V -> VOL_OUT_R
- C36 pad 2: GND -> Net-(C36-Pad2)
- C37 pad 2: AUDIO_OUT_L -> AUDIO_OUT_R
- C7 pad 1: +15V -> Net-(C7-Pad1)
- C7 pad 2: GND -> VOL_OUT_L
- C8 pad 1: +15V -> Net-(C8-Pad1)
- C8 pad 2: GND -> VOL_OUT_R
- C9 pad 1: Net-(C9-Pad1) -> +15V
- C9 pad 2: VOL_OUT_L -> GND
- R1 pad 2: Net-(C2-Pad1) -> Net-(C1-Pad1)
- R10 pad 2: Net-(C10-Pad1) -> Net-(C8-Pad1)
- R11 pad 1: Net-(C9-Pad1) -> Net-(C7-Pad1)
- R12 pad 1: Net-(C10-Pad1) -> Net-(C8-Pad1)
- R18 pad 1: Net-(C6-Pad2) -> Net-(R18-Pad1)
- R18 pad 2: VBIAS_R -> VBIAS_L
- R19 pad 2: VBIAS_L -> VBIAS_R
- R2 pad 2: Net-(C3-Pad1) -> Net-(C2-Pad1)
- R20 pad 1: Net-(R20-Pad1) -> Net-(C6-Pad2)
- R27 pad 1: Net-(C17-Pad2) -> Net-(C21-Pad1)
- R27 pad 2: VBIAS_L -> Net-(R21-Pad2)
- R28 pad 1: Net-(C18-Pad2) -> Net-(C22-Pad1)
- R28 pad 2: VBIAS_R -> Net-(R22-Pad2)
- R29 pad 1: Net-(C23-Pad1) -> Net-(C21-Pad2)
- R29 pad 2: Net-(R21-Pad2) -> L_Pot3
- R30 pad 1: LEFT_AUDIO_IN -> Net-(C22-Pad2)
- R30 pad 2: Net-(C17-Pad1) -> R_Pot3
- R31 pad 1: RIGHT_AUDIO_IN -> Net-(C17-Pad2)
- R31 pad 2: Net-(C18-Pad1) -> VBIAS_L
- R32 pad 1: Net-(C24-Pad1) -> Net-(C18-Pad2)
- R32 pad 2: Net-(R22-Pad2) -> VBIAS_R
- R33 pad 1: Net-(C23-Pad2) -> LEFT_AUDIO_IN
- R33 pad 2: L_Pot3 -> Net-(C17-Pad1)
- R34 pad 1: Net-(R34-Pad1) -> RIGHT_AUDIO_IN
- R34 pad 2: LEFT_BUF_AUDIO -> Net-(C18-Pad1)
- R35 pad 1: Net-(R35-Pad1) -> Net-(C21-Pad1)
- R35 pad 2: RIGHT_BUF_AUDIO -> Net-(C21-Pad2)
- R36 pad 1: Net-(C24-Pad2) -> Net-(C22-Pad1)
- R36 pad 2: R_Pot3 -> Net-(C22-Pad2)
- R37 pad 1: GND -> Net-(R37-Pad1)
- R37 pad 2: Net-(C17-Pad1) -> LEFT_BUF_AUDIO
- R38 pad 1: GND -> Net-(R38-Pad1)
- R38 pad 2: Net-(C18-Pad1) -> RIGHT_BUF_AUDIO
- R39 pad 1: Net-(C23-Pad1) -> GND
- R39 pad 2: Net-(C23-Pad2) -> Net-(C17-Pad1)
- R40 pad 1: Net-(C24-Pad1) -> GND
- R40 pad 2: Net-(C24-Pad2) -> Net-(C18-Pad1)
- R46 pad 2: POWER_AMP_IN_L -> POWER_AMP_OUT_L
- R48 pad 2: POWER_AMP_OUT_L -> POWER_AMP_IN_L
- R49 pad 1: Net-(R49-Pad1) -> POWER_AMP_OUT_L
- R49 pad 2: POWER_AMP_IN_L -> Net-(C26-Pad1)
- R50 pad 1: Net-(R50-Pad1) -> GND
- R50 pad 2: POWER_AMP_OUT_L -> AUDIO_OUT_L
- R54 pad 1: Net-(C31-Pad2) -> Net-(R54-Pad1)
- R54 pad 2: VBIAS_R -> POWER_AMP_OUT_L
- R55 pad 2: POWER_AMP_OUT_R -> POWER_AMP_IN_L
- R56 pad 2: POWER_AMP_OUT_R -> POWER_AMP_OUT_L
- R57 pad 2: POWER_AMP_IN_R -> POWER_AMP_OUT_L
- R58 pad 2: POWER_AMP_OUT_R -> POWER_AMP_OUT_L
- R60 pad 2: POWER_AMP_IN_R -> POWER_AMP_OUT_L
- R61 pad 2: POWER_AMP_OUT_R -> POWER_AMP_OUT_L
- R62 pad 2: POWER_AMP_OUT_R -> POWER_AMP_OUT_L
- R64 pad 1: Net-(R64-Pad1) -> Net-(C36-Pad2)
- R64 pad 2: POWER_AMP_OUT_R -> VBIAS_R
- R66 pad 1: GND -> Net-(R66-Pad1)
- R66 pad 2: AUDIO_OUT_L -> POWER_AMP_OUT_R
- R67 pad 1: POWER_AMP_OUT_R -> Net-(R67-Pad1)
- R67 pad 2: Net-(C38-Pad1) -> POWER_AMP_OUT_R
- R68 pad 1: GND -> Net-(R68-Pad1)
- R68 pad 2: AUDIO_OUT_R -> POWER_AMP_OUT_R
- R7 pad 1: L_Pot3 -> Net-(C1-Pad1)
- R7 pad 2: Net-(C9-Pad1) -> GND
- R9 pad 1: Net-(C3-Pad1) -> L_Pot3
- R9 pad 2: GND -> Net-(C7-Pad1)
- U1 pad 3: Net-(C2-Pad1) -> Net-(C1-Pad1)
- U1 pad 5: Net-(C2-Pad1) -> Net-(C1-Pad1)
- U1 pad 6: Net-(R19-Pad1) -> Net-(R18-Pad1)
- U1 pad 7: Net-(R19-Pad1) -> Net-(R18-Pad1)
- U10 pad 6: Net-(R48-Pad1) -> Net-(R52-Pad1)
- U10 pad 7: Net-(R48-Pad1) -> Net-(R52-Pad1)
- U11 pad 3: Net-(C25-Pad2) -> POWER_AMP_IN_L
- U11 pad 5: Net-(C25-Pad2) -> POWER_AMP_IN_L
- U11 pad 6: Net-(R49-Pad1) -> Net-(R53-Pad1)
- U11 pad 7: Net-(R49-Pad1) -> Net-(R53-Pad1)
- U12 pad 1: Net-(R50-Pad1) -> Net-(R47-Pad1)
- U12 pad 2: Net-(R50-Pad1) -> Net-(R47-Pad1)
- U12 pad 6: Net-(R52-Pad1) -> Net-(R54-Pad1)
- U12 pad 7: Net-(R52-Pad1) -> Net-(R54-Pad1)
- U13 pad 1: Net-(R51-Pad1) -> Net-(R48-Pad1)
- U13 pad 2: Net-(R51-Pad1) -> Net-(R48-Pad1)
- U13 pad 3: POWER_AMP_IN_L -> Net-(C25-Pad2)
- U13 pad 5: POWER_AMP_IN_L -> Net-(C25-Pad2)
- U13 pad 6: Net-(R53-Pad1) -> Net-(R55-Pad1)
- U13 pad 7: Net-(R53-Pad1) -> Net-(R55-Pad1)
- U14 pad 1: Net-(R55-Pad1) -> Net-(R56-Pad1)
- U14 pad 2: Net-(R55-Pad1) -> Net-(R56-Pad1)
- U14 pad 3: POWER_AMP_IN_R -> POWER_AMP_IN_L
- U14 pad 5: POWER_AMP_IN_R -> POWER_AMP_IN_L
- U14 pad 6: Net-(R58-Pad1) -> Net-(R60-Pad1)
- U14 pad 7: Net-(R58-Pad1) -> Net-(R60-Pad1)
- U15 pad 1: Net-(R56-Pad1) -> Net-(R57-Pad1)
- U15 pad 2: Net-(R56-Pad1) -> Net-(R57-Pad1)
- U15 pad 3: POWER_AMP_IN_R -> POWER_AMP_IN_L
- U15 pad 5: POWER_AMP_IN_R -> POWER_AMP_IN_L
- U15 pad 6: Net-(R59-Pad1) -> Net-(R61-Pad1)
- U15 pad 7: Net-(R59-Pad1) -> Net-(R61-Pad1)
- U16 pad 1: Net-(R57-Pad1) -> Net-(R58-Pad1)
- U16 pad 2: Net-(R57-Pad1) -> Net-(R58-Pad1)
- U16 pad 3: Net-(C31-Pad2) -> POWER_AMP_IN_L
- U16 pad 5: Net-(C31-Pad2) -> POWER_AMP_IN_L
- U16 pad 6: Net-(R60-Pad1) -> Net-(R62-Pad1)
- U16 pad 7: Net-(R60-Pad1) -> Net-(R62-Pad1)
- U2 pad 3: Net-(C3-Pad1) -> Net-(C2-Pad1)
- U2 pad 5: Net-(C3-Pad1) -> Net-(C2-Pad1)
- U2 pad 6: Net-(R20-Pad1) -> Net-(R19-Pad1)
- U2 pad 7: Net-(R20-Pad1) -> Net-(R19-Pad1)
- U3 pad 1: Net-(R34-Pad1) -> Net-(R21-Pad2)
- U3 pad 2: Net-(R34-Pad1) -> Net-(R21-Pad2)
- U3 pad 3: Net-(C17-Pad2) -> Net-(C5-Pad2)
- U3 pad 5: Net-(C17-Pad2) -> Net-(R3-Pad2)
- U3 pad 6: Net-(R41-Pad1) -> Net-(C7-Pad1)
- U3 pad 7: Net-(R41-Pad1) -> VOL_OUT_L
- U4 pad 1: Net-(R35-Pad1) -> Net-(R22-Pad2)
- U4 pad 2: Net-(R35-Pad1) -> Net-(R22-Pad2)
- U4 pad 3: Net-(C18-Pad2) -> Net-(C6-Pad2)
- U4 pad 5: Net-(C18-Pad2) -> Net-(R4-Pad2)
- U4 pad 6: Net-(R42-Pad1) -> Net-(C8-Pad1)
- U4 pad 7: Net-(R42-Pad1) -> VOL_OUT_R
- U5 pad 1: Net-(R21-Pad2) -> Net-(C21-Pad2)
- U5 pad 2: Net-(R21-Pad2) -> Net-(C21-Pad1)
- U5 pad 3: Net-(C5-Pad2) -> Net-(R13-Pad2)
- U5 pad 5: Net-(R3-Pad2) -> Net-(R14-Pad1)
- U5 pad 6: Net-(C9-Pad1) -> Net-(C11-Pad1)
- U5 pad 7: VOL_OUT_L -> Net-(C11-Pad2)
- U6 pad 1: Net-(C23-Pad2) -> Net-(C22-Pad2)
- U6 pad 2: Net-(C23-Pad1) -> Net-(C22-Pad1)
- U6 pad 3: Net-(R13-Pad2) -> Net-(R15-Pad2)
- U6 pad 5: Net-(R14-Pad1) -> Net-(R16-Pad1)
- U6 pad 6: Net-(C11-Pad1) -> Net-(C12-Pad1)
- U6 pad 7: Net-(C11-Pad2) -> Net-(C12-Pad2)
- U7 pad 1: Net-(R22-Pad2) -> Net-(R37-Pad1)
- U7 pad 2: Net-(R22-Pad2) -> Net-(R37-Pad1)
- U7 pad 3: Net-(C6-Pad2) -> Net-(C17-Pad2)
- U7 pad 5: Net-(R4-Pad2) -> Net-(C17-Pad2)
- U7 pad 6: Net-(C10-Pad1) -> Net-(R41-Pad1)
- U7 pad 7: VOL_OUT_R -> Net-(R41-Pad1)
- U8 pad 1: Net-(C24-Pad2) -> Net-(R38-Pad1)
- U8 pad 2: Net-(C24-Pad1) -> Net-(R38-Pad1)
- U8 pad 3: Net-(R15-Pad2) -> Net-(C18-Pad2)
- U8 pad 5: Net-(R16-Pad1) -> Net-(C18-Pad2)
- U8 pad 6: Net-(C12-Pad1) -> Net-(R42-Pad1)
- U8 pad 7: Net-(C12-Pad2) -> Net-(R42-Pad1)
Routing:
- net VBIAS_L: track 2.29 -> 157.0 mm, vias 0 -> 3
- net +15V: track 5.49 -> 154.9 mm, vias 0 -> 9
- net GND: track 10.2 -> 131.1 mm, vias 0 -> 50
- net VBIAS_R: track 2.29 -> 120.2 mm, vias 0 -> 5
- net POWER_AMP_IN_L: track 0.00 -> 68.0 mm
- net R_Pot2: track 0.00 -> 53.2 mm, vias 0 -> 1
- net POWER_AMP_IN_R: track 0.00 -> 50.1 mm
- net Net-(C18-Pad2): track 0.00 -> 49.3 mm, vias 0 -> 2
- net R_Pot1: track 0.00 -> 49.2 mm
- net Net-(C17-Pad2): track 0.00 -> 46.9 mm
- net R_Pot3: track 0.00 -> 45.5 mm
- net L_Pot1: track 0.00 -> 41.9 mm
- net POWER_AMP_OUT_L: track 0.00 -> 40.7 mm
- net POWER_AMP_OUT_R: track 0.00 -> 40.5 mm
- net RIGHT_AUDIO_IN: track 0.00 -> 35.4 mm
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Other:
- board outline added: 110 x 76.5 mm
- copper layers 2 -> 4

Commit message: pcb layout complete
Parts:
- moved C31 3.57 mm to (93.6, 82.9), turned to 180 degrees
- moved R69 0.65 mm to (129.8, 88.4)
- moved R76 0.65 mm to (128.0, 88.4)
- moved R71 0.28 mm to (120.8, 107.2), turned to 0 degrees
- moved J1 0.23 mm to (146.0, 54.2)
Routing:
- net +15V: track 154.9 -> 365.4 mm, vias 9 -> 26
- net L_Pot2: track 0.00 -> 104.6 mm, vias 0 -> 1
- net L_Pot3: track 9.73 -> 110.7 mm, vias 0 -> 1
- net VBIAS_R: track 120.2 -> 154.4 mm, vias 5 -> 6
- net POWER_AMP_IN_R: track 50.1 -> 72.6 mm
- net Net-(C36-Pad2): track 30.7 -> 24.9 mm, vias 0 -> 2
- net VBIAS_L: track 157.0 -> 151.8 mm
- net Net-(R69-Pad1): track 1.27 -> 5.06 mm
- net GND: track 131.1 -> 134.9 mm
- net Net-(C37-Pad1): track 28.6 -> 27.1 mm
- net AUDIO_OUT_R: track 28.9 -> 30.2 mm
- net VOL_OUT_R: track 29.0 -> 28.2 mm
- net Net-(R76-Pad1): track 11.2 -> 11.9 mm
- net Net-(R21-Pad2): track 18.6 -> 19.3 mm
- net L_Pot1: track 41.9 -> 41.4 mm
- added copper zone on B.Cu, net GND
- added copper zone on F.Cu, net GND
Other:
- board size 110 x 76.5 mm -> 110 x 72 mm

Commit message: updated files
Parts:
- moved C4 3.97 mm to (177.5, 68.4)
- moved C20 3.00 mm to (168.2, 68.1)
- moved R34 3.00 mm to (169.6, 67.6)
- moved R38 3.00 mm to (172.2, 64.3)
- moved R40 3.00 mm to (172.2, 68.4)
- moved R42 3.00 mm to (172.2, 66.3)
- moved C24 2.62 mm to (171.0, 54.2)
- moved R32 2.62 mm to (174.0, 53.4)
- moved U8 2.62 mm to (172.2, 59.2)
- moved C19 2.62 mm to (160.1, 68.5)
- moved C23 2.62 mm to (161.6, 54.5)
- moved R33 2.62 mm to (161.5, 68.0)
- moved R37 2.62 mm to (164.2, 64.7)
- moved R39 2.62 mm to (164.2, 68.8)
- moved R41 2.62 mm to (164.2, 66.7)
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Routing:
- net Net-(C18-Pad2): track 49.3 -> 13.3 mm, vias 2 -> 0
- net RIGHT_AUDIO_IN: track 35.4 -> 17.5 mm
- net VBIAS_R: track 154.4 -> 138.1 mm, vias 6 -> 8
- net +15V: track 365.4 -> 349.7 mm
- net VBIAS_L: track 151.8 -> 139.8 mm, vias 3 -> 5
- net LEFT_AUDIO_IN: track 21.1 -> 9.72 mm
- net RIGHT_BUF_AUDIO: track 8.47 -> 2.03 mm
- net Net-(C17-Pad1): track 8.02 -> 3.33 mm
- net Net-(C18-Pad1): track 7.72 -> 3.45 mm
- net L_Pot1: track 41.4 -> 44.6 mm
- net LEFT_BUF_AUDIO: track 12.1 -> 8.88 mm
- net Net-(R42-Pad1): track 11.1 -> 13.7 mm, vias 2 -> 0
- net Net-(C17-Pad2): track 46.9 -> 48.9 mm
- net R_Pot1: track 49.2 -> 47.7 mm
- net VOL_OUT_R: track 28.2 -> 27.5 mm
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Other:
- outline, holes or cut-outs redrawn
