File: AMP/AMP.kicad_sch (KiCad schematic)
At the start: 53 parts, among them U1 NE5532, U2 NE5532, U3 NE5532, U4 NE5532, U5 NE5532, U6 NE5532

Commit message: amp updated files
Parts:
- added C?: 10u, symbol Device:C_Small
- added C? (x3): 100p, symbol Device:C_Small
- added C?: 220u, symbol Device:C_Polarized_Small
- added C? (x2): 100n, symbol Device:C_Small
- added R? (x3): 5.6k, symbol Device:R_Small
- added R?: 47k, symbol Device:R_Small
- added R? (x6): 1k, symbol Device:R_Small
- added R?: 3.3k, symbol Device:R_Small
- added R? (x2): 10, symbol Device:R_Small
- added U? (x6): NE5532, symbol Amplifier_Operational:NE5532
Connections:
- net RIGHT_BUF_AUDIO: now also C?.1
- net VBIAS_L: now also R?.1
- net VBIAS_R: now also R?.1, R?.1, R?.2, R?.2
- net R_Pot3: now reaches RV?.4
- net R_Pot3: now also R?.1, R?.2, R?.2
- net R_Pot2: now reaches RV?.5
- net R_Pot2: now also C?.1
- net R_Pot1: now reaches RV?.6
- net R_Pot1: now also C?.2
- net VOL_OUT_L: now reaches C?.2, R?.2, U5.7
- net at U5.5 (+): now also R?.2
- new net: C?.1, R?.1, R?.1, U?.2 (-)
- new net: C?.2, R?.1, R?.2, U?.1
- new net: C?.2, R?.1, U?.3 (+)
- new net: C?.1, R?.1, R?.1, U?.6 (-)
- new net: C?.2, R?.1, R?.2, U?.7
- new net: R?.1, U?.5 (+)
- new net: R?.2, U?.3 (+)
- new net: C?.1, R?.1, R?.2, U?.6 (-)
- new net: R?.2, R?.2, U?.1, U?.2 (-)
- new net: C?.2, U?.4 (V-) (x2)
- new net: C?.1, U?.8 (V+) (x2)
- new net: R?.2, U?.5 (+)
- new net VOL_OUT_R: C?.2, R?.2, U?.7
Other:
- note added: "Volume Control (LEFT)"
- note added: "Volume Control (RIGHT)"
- note removed: "Volume Control"
- moved on the sheet: C?, R?, RV?, U1A, U1B, U1C, U2A, U2B, U2C, U3A, U3B, U3C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

Commit message: amp updated files
Parts:
- added C? (x18): 100n, symbol Device:C_Small
- added C? (x2): 10u, symbol Device:C_Small
- added R? (x16): 1, symbol Device:R_Small
- added R? (x2): 10k, symbol Device:R_Small
- added R? (x4): 10, symbol Device:R_Small
- added U? (x30): NE5532, symbol Amplifier_Operational:NE5532
- gave numbers to parts that had none: 2
Connections:
- net VBIAS_L: now also R?.2
- net VBIAS_R: now also R?.2
- net VOL_OUT_L: now also C?.1
- net VOL_OUT_R: now also C?.1
- new net: C?.1, U?.3 (+), U?.5 (+) (x8)
- new net: R?.1, U?.6 (-), U?.7 (x10)
- new net: C?.1, U?.8 (V+) (x10)
- new net: C?.2, U?.4 (V-) (x10)
- new net: R?.1, U?.1, U?.2 (-) (x10)
- new net: C?.2, R?.1, U?.3 (+), U?.5 (+) (x2)
- new net POWER_AMP_IN_L: C?.2, C?.2, C?.2, C?.2, R?.2, R?.2
- new net POWER_AMP_IN_R: C?.2, C?.2, C?.2, C?.2, R?.2, R?.2
- new net POWER_AMP_OUT_L: R?.2, R?.2, R?.2, R?.2, R?.2, R?.2, R?.2, R?.2
- new net POWER_AMP_OUT_R: R?.2, R?.2, R?.2, R?.2, R?.2, R?.2, R?.2, R?.2
Other:
- note added: "Baxandall Input Buffer (LEFT)"
- note added: "Baxandall Input Buffer (RIGHT)"
- note added: "Power Driver (LEFT)"
- note added: "Power Driver (RIGHT)"
- note added: "Pre-Driver (LEFT)"
- note added: "Pre-Driver (RIGHT)"
- note removed: "Input Buffer (LEFT)"
- note removed: "Input Buffer (RIGHT)"
- moved on the sheet: C?, R?, RV?, U5A, U5B, U5C, U6A, U6B, U6C, U7A, U7B, U7C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

Commit message: amp updated files
Parts:
- removed C? (x8): 100n, symbol Device:C_Small
- gave numbers to parts that had none: 111
Connections:
- net POWER_AMP_IN_L: now also U10.3 (+), U10.5 (+), U12.3 (+), U12.5 (+), U13.3 (+), U13.5 (+), U9.3 (+), U9.5 (+)
- net POWER_AMP_IN_R: now also U14.3 (+), U14.5 (+), U15.3 (+), U15.5 (+), U17.3 (+), U17.5 (+), U18.3 (+), U18.5 (+)
Other:
- moved on the sheet: C1, C10, C11, C12, C13, C14, C15, C16, C23, C24, C25, C26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

Commit message: schematic done
Parts:
- added C37, C38: 2200u, Capacitor_THT:CP_Radial_D12.5mm_P5.00mm, symbol Device:C_Polarized_Small
- added R65, R67: 10, Resistor_SMD:R_0603_1608Metric, symbol Device:R_Small
- added R66, R68: 10k, Resistor_SMD:R_1206_3216Metric, symbol Device:R_Small
- C1, C4: footprint (none) -> Capacitor_THT:CP_Radial_D6.3mm_P2.50mm; LCSC (none) -> C2831780
- C10, C11, C12, C23, C24, C9: footprint (none) -> Resistor_SMD:R_0603_1608Metric; LCSC (none) -> C14858
- C13, C14, C15, C16, C21, C22, C26, C27, C28, C29, C30, C32, C33, C34, C35, C36, C7, C8: footprint (none) -> Resistor_SMD:R_0603_1608Metric; LCSC (none) -> C14663
- C17, C18: footprint (none) -> Capacitor_THT:C_Rect_L24.0mm_W12.8mm_P22.50mm_MKT; LCSC (none) -> C3019077
- C19, C20: footprint (none) -> Capacitor_SMD:C_0201_0603Metric; LCSC (none) -> C1588
- C2, C3, C5, C6: footprint (none) -> Resistor_SMD:R_0603_1608Metric; LCSC (none) -> C96446
- C25, C31: footprint (none) -> Capacitor_THT:C_Axial_L22.0mm_D10.5mm_P27.50mm_Horizontal; LCSC (none) -> C5116053
- R1, R2, R8, R9: footprint (none) -> Resistor_THT:R_Axial_DIN0516_L15.5mm_D5.0mm_P20.32mm_Horizontal; LCSC (none) -> C714455
- R10, R7: footprint (none) -> Resistor_SMD:R_1206_3216Metric; LCSC (none) -> C706452
- R11, R12, R25, R26, R39, R40: footprint (none) -> Resistor_SMD:R_0603_1608Metric; LCSC (none) -> C445632
- R13, R14, R15, R16, R21, R22, R29, R3, R32, R4: footprint (none) -> Resistor_SMD:R_0603_1608Metric; LCSC (none) -> C110776
- R17, R18: footprint (none) -> Resistor_SMD:R_0603_1608Metric; LCSC (none) -> C307918
- R19, R20, R23, R24, R33, R34, R35, R36, R41, R42, R46, R49, R5, R57, R6, R60: footprint (none) -> Resistor_SMD:R_0603_1608Metric; LCSC (none) -> C319922
- R27, R28, R37, R38: footprint (none) -> Resistor_SMD:R_0603_1608Metric; LCSC (none) -> C375508
- R30, R31: footprint (none) -> Resistor_SMD:R_0603_1608Metric; LCSC (none) -> C217683
- R43, R54: footprint (none) -> Resistor_SMD:R_1206_3216Metric; LCSC (none) -> C406727
- R44, R45, R47, R48, R50, R51, R52, R53, R55, R56, R58, R59, R61, R62, R63, R64: footprint (none) -> Resistor_SMD:R_1206_3216Metric; LCSC (none) -> C111291
- U1, U10, U11, U12, U13, U14, U15, U16, U17, U18, U2, U3, U4, U5, U6, U7, U8, U9: footprint (none) -> AUDIO_ECAD:NE5532DR; LCSC (none) -> C7426
Connections:
- net GND: now also R66.1, R68.1
- net POWER_AMP_OUT_L: now also R65.1
- net POWER_AMP_OUT_R: now also R67.1
- new net: C37.1, R65.2
- new net: C38.1, R67.2
- new net AUDIO_OUT_L: C37.2, R66.2
- new net AUDIO_OUT_R: C38.2, R68.2
Other:
- note added: "Output Protection & Filtering (LEFT)"
- moved on the sheet: C25, C26, C27, C28, C29, C30, C31, C32, C33, C34, C35, C36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

Commit message: amp updated files
Parts:
- added J1, J3: AudioJack4, Connector_Audio:Jack_3.5mm_PJ320D_Horizontal, symbol Connector:AudioJack4
- added J2: Screw_Terminal_01x02, TerminalBlock:TerminalBlock_Altech_AK300-2_P5.00mm, symbol Connector:Screw_Terminal_01x02
Connections:
- net +15V: now also C13.1, C14.1, C15.1, C16.1, C21.1, C22.1, C26.1, C27.1, C28.1, C29.1, C30.1, C32.1, C33.1, C34.1, C35.1, C36.1, C7.1, C8.1, U1.8 (V+), U10.8 (V+), U11.8 (V+), U12.8 (V+), U13.8 (V+), U14.8 (V+), U15.8 (V+), U16.8 (V+), U17.8 (V+), U18.8 (V+), U2.8 (V+), U3.8 (V+), U4.8 (V+), U5.8 (V+), U6.8 (V+), U7.8 (V+), U8.8 (V+), U9.8 (V+), J2.1 (Pin_1)
- net AUDIO_OUT_L: now also J3.T
- net AUDIO_OUT_R: now also J3.R1
- net GND: now also C13.2, C14.2, C15.2, C16.2, C21.2, C22.2, C26.2, C27.2, C28.2, C29.2, C30.2, C32.2, C33.2, C34.2, C35.2, C36.2, C7.2, C8.2, U1.4 (V-), U10.4 (V-), U11.4 (V-), U12.4 (V-), U13.4 (V-), U14.4 (V-), U15.4 (V-), U16.4 (V-), U17.4 (V-), U18.4 (V-), U2.4 (V-), U3.4 (V-), U4.4 (V-), U5.4 (V-), U6.4 (V-), U7.4 (V-), U8.4 (V-), U9.4 (V-), J1.S, J2.2 (Pin_2), J3.S
- net LEFT_AUDIO_IN: now also J1.R1
- net RIGHT_AUDIO_IN: now also J1.T
- no-connect marks 0 -> 2
Other:
- moved on the sheet: C13, C14, C15, C16, C17, C18, C19, C20, C21, C22, C25, C26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

Commit message: pcb layout
Parts:
- R1, R2, R8, R9: footprint Resistor_THT:R_Axial_DIN0516_L15.5mm_D5.0mm_P20.32mm_Horizontal -> Resistor_SMD:R_0603_1608Metric; LCSC C714455 -> C114662
Connections:
- net LEFT_AUDIO_IN: now also J1.T; no longer J1.R1
- net RIGHT_AUDIO_IN: now also J1.R1; no longer J1.T
Changed lines of the file:
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@@
     )
   )
-  (global_label "RIGHT_AUDIO_IN" (shape input) (at 433.07 205.74 0) (fields_autoplaced)
-    (effects (font (size 1.27 1.27)) (justify left))
-    (property "Intersheet References" "${INTERSHEET_REFS}" (id 0) (at 450.4207 205.6606 0)
-      (effects (font (size 1.27 1.27)) (justify left) hide)
-    )
-  )
   (global_label "VOL_OUT_R" (shape input) (at 557.53 50.8 0) (fields_autoplaced)
     (effects (font (size 1.27 1.27)) (justify left))
@@
     )
   )
+  (global_label "RIGHT_AUDIO_IN" (shape input) (at 433.07 203.2 0) (fields_autoplaced)
+    (effects (font (size 1.27 1.27)) (justify left))
+    (property "Intersheet References" "${INTERSHEET_REFS}" (id 0) (at 450.4207 203.1206 0)
+      (effects (font (size 1.27 1.27)) (justify left) hide)
+    )
+  )
   (global_label "POWER_AMP_OUT_L" (shape input) (at 184.15 237.49 0) (fields_autoplaced)
     (effects (font (size 1.27 1.27)) (justify left))
@@
     )
   )
+  (global_label "LEFT_AUDIO_IN" (shape input) (at 433.07 205.74 0) (fields_autoplaced)
+    (effects (font (size 1.27 1.27)) (justify left))
+    (property "Intersheet References" "${INTERSHEET_REFS}" (id 0) (at 449.2112 205.8194 0)
+      (effects (font (size 1.27 1.27)) (justify left) hide)
+    )
+  )
   (global_label "POWER_AMP_IN_L" (shape input) (at 228.6 186.69 180) (fields_autoplaced)
     (effects (font (size 1.27 1.27)) (justify right))
@@
     )
   )
-  (global_label "LEFT_AUDIO_IN" (shape input) (at 433.07 203.2 0) (fields_autoplaced)
-    (effects (font (size 1.27 1.27)) (justify left))
-    (property "Intersheet References" "${INTERSHEET_REFS}" (id 0) (at 449.2112 203.2794 0)
-      (effects (font (size 1.27 1.27)) (justify left) hide)
-    )
-  )
   (global_label "VBIAS_L" (shape input) (at 279.4 69.85 180) (fields_autoplaced)
     (effects (font (size 1.27 1.27)) (justify right))
@@
       (effects (font (size 1.27 1.27)) (justify left))
     )
-    (property "Footprint" "Resistor_THT:R_Axial_DIN0516_L15.5mm_D5.0mm_P20.32mm_Horizontal" (id 2) (at 27.94 43.18 0)
+    (property "Footprint" "Resistor_SMD:R_0603_1608Metric" (id 2) (at 27.94 43.18 0)
       (effects (font (size 1.27 1.27)) hide)
     )
-    (property "Datasheet" "~" (id 3) (at 27.94 43.18 0)
+    (property "Datasheet" "https://datasheet.lcsc.com/lcsc/2304140030_YAGEO-RC0603FR-072K2L_C114662.pdf" (id 3) (at 27.94 43.18 0)
       (effects (font (size 1.27 1.27)) hide)
     )
-    (property "LCSC" "C714455" (id 4) (at 27.94 43.18 0)
+    (property "LCSC" "C114662" (id 4) (at 27.94 43.18 0)
       (effects (font (size 1.27 1.27)) hide)
     )
@@
       (effects (font (size 1.27 1.27)) (justify left))
     )
-    (property "Footprint" "Resistor_THT:R_Axial_DIN0516_L15.5mm_D5.0mm_P20.32mm_Horizontal" (id 2) (at 116.84 43.18 0)
+    (property "Footprint" "Resistor_SMD:R_0603_1608Metric" (id 2) (at 116.84 43.18 0)
       (effects (font (size 1.27 1.27)) hide)
     )
-    (property "Datasheet" "~" (id 3) (at 116.84 43.18 0)
+    (property "Datasheet" "https://datasheet.lcsc.com/lcsc/2304140030_YAGEO-RC0603FR-072K2L_C114662.pdf" (id 3) (at 116.84 43.18 0)
       (effects (font (size 1.27 1.27)) hide)
     )
-    (property "LCSC" "C714455" (id 4) (at 116.84 43.18 0)
+    (property "LCSC" "C114662" (id 4) (at 116.84 43.18 0)
       (effects (font (size 1.27 1.27)) hide)
     )
@@
       (effects (font (size 1.27 1.27)) (justify left))
     )
-    (property "Footprint" "Resistor_THT:R_Axial_DIN0516_L15.5mm_D5.0mm_P20.32mm_Horizontal" (id 2) (at 27.94 53.34 0)
+    (property "Footprint" "Resistor_SMD:R_0603_1608Metric" (id 2) (at 27.94 53.34 0)
       (effects (font (size 1.27 1.27)) hide)
     )
-    (property "Datasheet" "~" (id 3) (at 27.94 53.34 0)
+    (property "Datasheet" "https://datasheet.lcsc.com/lcsc/2304140030_YAGEO-RC0603FR-072K2L_C114662.pdf" (id 3) (at 27.94 53.34 0)
       (effects (font (size 1.27 1.27)) hide)
     )
-    (property "LCSC" "C714455" (id 4) (at 27.94 53.34 0)
+    (property "LCSC" "C114662" (id 4) (at 27.94 53.34 0)
       (effects (font (size 1.27 1.27)) hide)
     )
@@
       (effects (font (size 1.27 1.27)) (justify left))
     )
-    (property "Footprint" "Resistor_THT:R_Axial_DIN0516_L15.5mm_D5.0mm_P20.32mm_Horizontal" (id 2) (at 116.84 53.34 0)
+    (property "Footprint" "Resistor_SMD:R_0603_1608Metric" (id 2) (at 116.84 53.34 0)
       (effects (font (size 1.27 1.27)) hide)
     )
-    (property "Datasheet" "~" (id 3) (at 116.84 53.34 0)
+    (property "Datasheet" "https://datasheet.lcsc.com/lcsc/2304140030_YAGEO-RC0603FR-072K2L_C114662.pdf" (id 3) (at 116.84 53.34 0)
       (effects (font (size 1.27 1.27)) hide)
     )
-    (property "LCSC" "C714455" (id 4) (at 116.84 53.34 0)
+    (property "LCSC" "C114662" (id 4) (at 116.84 53.34 0)
       (effects (font (size 1.27 1.27)) hide)
     )
@@
     )
     (path "/200c63d5-9f0c-4606-917d-24a8280ed9ed"
-      (reference "R1") (unit 1) (value "2.2k") (footprint "Resistor_THT:R_Axial_DIN0516_L15.5mm_D5.0mm_P20.32mm_Horizontal")
+      (reference "R1") (unit 1) (value "2.2k") (footprint "Resistor_SMD:R_0603_1608Metric")
     )
     (path "/e1a0cc3c-2cac-4d0a-abe1-d80d5486209e"
-      (reference "R2") (unit 1) (value "2.2k") (footprint "Resistor_THT:R_Axial_DIN0516_L15.5mm_D5.0mm_P20.32mm_Horizontal")
+      (reference "R2") (unit 1) (value "2.2k") (footprint "Resistor_SMD:R_0603_1608Metric")
     )
     (path "/0d0a4ca1-a81c-40e5-aa87-699cf3e69320"
@@
     )
     (path "/f6de87ba-476e-4789-9f15-f77e20cfa9a4"
-      (reference "R8") (unit 1) (value "2.2k") (footprint "Resistor_THT:R_Axial_DIN0516_L15.5mm_D5.0mm_P20.32mm_Horizontal")
+      (reference "R8") (unit 1) (value "2.2k") (footprint "Resistor_SMD:R_0603_1608Metric")
     )
     (path "/f91a8d3f-d2a2-418e-a962-86afff331ba8"
-      (reference "R9") (unit 1) (value "2.2k") (footprint "Resistor_THT:R_Axial_DIN0516_L15.5mm_D5.0mm_P20.32mm_Horizontal")
+      (reference "R9") (unit 1) (value "2.2k") (footprint "Resistor_SMD:R_0603_1608Metric")
     )
     (path "/3d156a46-95e7-451b-88f8-4f39928bd8e1"

Commit message: updated files
Parts:
- removed C26, C32: 100n, Resistor_SMD:R_0603_1608Metric, symbol Device:C_Small
- removed R44, R55: 1, Resistor_SMD:R_1206_3216Metric, symbol Device:R_Small
- removed U14, U9: NE5532, AUDIO_ECAD:NE5532DR, symbol Amplifier_Operational:NE5532
- added C29, C30, C34, C40, C41, C45: 100n, Resistor_SMD:R_0603_1608Metric, symbol Device:C_Small
- added J4: Barrel_Jack_MountingPin, Connector_BarrelJack:BarrelJack_Horizontal, symbol Connector:Barrel_Jack_MountingPin
- added R46, R53, R54, R62, R67, R68, R74, R75, R79, R83: 1, Resistor_SMD:R_1206_3216Metric, symbol Device:R_Small
- added U11, U12, U16, U20, U21, U25: NE5532, AUDIO_ECAD:NE5532DR, symbol Amplifier_Operational:NE5532
- J3: renamed from J2; footprint TerminalBlock:TerminalBlock_Altech_AK300-2_P5.00mm -> TerminalBlock:TerminalBlock_bornier-2_P5.08mm; LCSC (none) -> C430601
- R1, R2: LCSC C114662 -> C557651
- R7: renamed from R8; LCSC C114662 -> C557651
- R8: renamed from R9; LCSC C114662 -> C557651
- RV1: footprint Potentiometer_THT:Potentiometer_Alpha_RD902F-40-00D_Dual_Vertical -> Potentiometer_THT:Potentiometer_Alps_RK163_Dual_Horizontal
- renumbered C2 to C1, C8 to C10, C15 to C13, C16 to C14, C13 to C15, C14 to C16, C3 to C2, C23 to C21, C24 to C22, C21 to C23, C22 to C24, C37 to C26, C27 to C28, C1 to C3, C28 to C31, C29 to C32, C30 to C33, C31 to C36, C38 to C37, C33 to C39, C34 to C42, C35 to C43, C36 to C44, C9 to C7, C10 to C8, C7 to C9, J3 to J2, R19 to R18, R20 to R19, R18 to R20, R29 to R27, R32 to R28, R33 to R29, R36 to R30, R27 to R31, R28 to R32, R30 to R33, R31 to R34, R39 to R35, R40 to R36, R34 to R37, R35 to R38, R37 to R39, R38 to R40, R46 to R48, R65 to R49, R66 to R50, R48 to R52, R49 to R55, R50 to R56, R51 to R57, R52 to R60, R53 to R61, R54 to R64, R56 to R66, R57 to R69, R67 to R70, R68 to R71, R59 to R73, R60 to R76, R61 to R77, R62 to R78, R63 to R81, R64 to R82, R7 to R9, U11 to U13, U12 to U14, U13 to U15, U15 to U19, U16 to U22, U17 to U23, U18 to U24, U5 to U3, U7 to U4, U6 to U5, U8 to U6, U3 to U7, U4 to U8
Connections:
- net +15V: now also C29.1, C30.1, C34.1, C40.1, C41.1, C45.1, J4.1, U11.8 (V+), U12.8 (V+), U16.8 (V+), U20.8 (V+), U21.8 (V+), U25.8 (V+)
- net GND: now also C29.2, C30.2, C34.2, C40.2, C41.2, C45.2, J4.2, J4.3 (MountPin), U11.4 (V-), U12.4 (V-), U16.4 (V-), U20.4 (V-), U21.4 (V-), U25.4 (V-)
- net POWER_AMP_IN_L: now also U11.3 (+), U11.5 (+), U12.3 (+), U12.5 (+), U16.3 (+), U16.5 (+)
- net POWER_AMP_IN_R: now also U20.3 (+), U20.5 (+), U21.3 (+), U21.5 (+), U25.3 (+), U25.5 (+)
- net POWER_AMP_OUT_L: now also R58.2, R46.2, R53.2, R54.2, R62.2
- net POWER_AMP_OUT_R: now also R67.2, R68.2, R74.2, R75.2, R79.2, R83.2; no longer R58.2
- net at R47.1: now also U12.1, U12.2 (-)
- net at R58.1: now also U16.1, U16.2 (-)
- new net: R74.1, U20.6 (-), U20.7
- new net: R67.1, U20.1, U20.2 (-)
- new net: R62.1, U16.6 (-), U16.7
- new net: R83.1, U25.6 (-), U25.7
- new net: R68.1, U21.1, U21.2 (-)
- new net: R46.1, U11.1, U11.2 (-)
- new net: R79.1, U25.1, U25.2 (-)
- new net: R54.1, U12.6 (-), U12.7
- new net: R53.1, U11.6 (-), U11.7
- new net: R75.1, U21.6 (-), U21.7
Other:
- note added: "Output Protection & Filtering (RIGHT)"
- moved on the sheet: C1, C10, C17, C18, C19, C2, C20, C23, C24, C25, C26, C28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

Commit message: updated files
Parts:
- removed C30: 100n, Resistor_SMD:R_0603_1608Metric, symbol Device:C_Small
- removed R47, R54: 1, Resistor_SMD:R_1206_3216Metric, symbol Device:R_Small
- removed U12: NE5532, AUDIO_ECAD:NE5532DR, symbol Amplifier_Operational:NE5532
- added C?: 100n, Resistor_SMD:R_0603_1608Metric, symbol Device:C_Small
- added R? (x2): 1, Resistor_SMD:R_1206_3216Metric, symbol Device:R_Small
- added U? (x3): NE5532, AUDIO_ECAD:NE5532DR, symbol Amplifier_Operational:NE5532
Connections:
- net +15V: now also C?.1, U?.8 (V+)
- net GND: now also C?.2, U?.4 (V-)
- net POWER_AMP_IN_L: now also U?.3 (+), U?.5 (+)
- net POWER_AMP_OUT_L: now also R?.2, R?.2
- new net: R?.1, U?.1, U?.2 (-)
- new net: R?.1, U?.6 (-), U?.7
Other:
- moved on the sheet: C26, C37, C41, R49, R50, R68, R70, R71, R75, U21A, U21B, U21C
